File: Minisumo_V1.brd (EAGLE design)
At the start: 70 x 95 mm, 57 parts, among them IC1 STM32H743VIT6NORMAL, J1 FTSH-107-01-L-DV-K-TR, Y1 ECS-3225MV

Commit message: 07_11_2021_15_50
Parts:
- moved C23 4.14 mm to (19.6, 48.1)
- moved C19 3.81 mm to (20.7, 48.1)
- moved C20 3.64 mm to (19.4, 55.1), turned to 270 degrees
- moved C17 1.02 mm to (38.0, 56.3)
- moved C16 1.02 mm to (38.0, 54.2)
Connections:
- net MD_CS1: now also IC1.68
- net MD_CS2: now also IC1.58
- net MD_DIS1: now also IC1.67
- net MD_DIS2: now also IC1.59
- net MD_IN1_PWM_A: now also IC1.63
- net MD_IN1_PWM_B: now also IC1.61
- net MD_IN2_DIR_A: now also IC1.64
- net MD_IN2_DIR_B: now also IC1.60
- net MD_NDIS: now also IC1.62
Routing:
- net MD_IN1_PWM_B: track 0.00 -> 22.3 mm, vias 0 -> 3
- net MD_IN2_DIR_B: track 0.00 -> 22.0 mm, vias 0 -> 3
- net MD_DIS2: track 0.00 -> 19.9 mm, vias 0 -> 3
- net MD_CS2: track 0.00 -> 19.9 mm, vias 0 -> 3
- net MD_NDIS: track 0.00 -> 18.6 mm, vias 0 -> 4
- net MD_DIS1: track 0.00 -> 12.5 mm, vias 0 -> 2
- net MD_CS1: track 0.00 -> 12.2 mm, vias 0 -> 2
- net MD_IN2_DIR_A: track 0.00 -> 8.72 mm, vias 0 -> 2
- net MD_IN1_PWM_A: track 0.00 -> 8.72 mm, vias 0 -> 2
- net N$16: track 0.00 -> 3.10 mm, vias 0 -> 1
- net SPI_MISO: track 27.3 -> 29.2 mm, vias 3 -> 4
- net TOF_GPIO2: track 68.7 -> 67.9 mm
- net XSHUT2: track 67.3 -> 67.9 mm
- net +3.3V: vias 7 -> 14
- added copper zone on layer 16, net MD_VS

Commit message: 07_11_2021_22_21
Parts:
- added U$4, U$5: MD_OUT, SamacSys_Parts:MD_OUT
- added U$6: BAT_POW, SamacSys_Parts:MD_OUT
- moved R6 4.67 mm to (3.17, 91.4), flipped to the top
- moved R5 1.83 mm to (67.3, 9.02)
- moved R7 1.40 mm to (1.91, 87.4), turned to 180 degrees
- moved SV2 1.02 mm to (3.43, 47.2)
- moved R9 0.85 mm to (64.6, 88.5)
- moved C18 0.28 mm to (32.8, 53.5)
- moved C21 0.25 mm to (35.7, 50.8)
- moved SV1 0.25 mm to (67.2, 47.2)
- moved C10 0.13 mm to (53.5, 48.2)
- moved C7 0.13 mm to (53.5, 46.1)
- moved C8 0.13 mm to (53.5, 47.2)
- moved C9 0.13 mm to (53.5, 45.1)
- moved J1 0.13 mm to (61.5, 46.5)
- moved C22 0.13 mm to (34.1, 53.5)
- turned CZ2 to 270 degrees
Connections:
- net GND: now also U$6.IN_2
- net MD_OUT1A: now also U$4.IN_1
- net MD_OUT1B: now also U$5.IN_1
- net MD_OUT2A: now also U$4.IN_2
- net MD_OUT2B: now also U$5.IN_2
- net TOF_GPIO3: now also IC1.37; no longer IC1.32
- net TOF_GPIO5: now also IC1.78
- net V_BAT: now also U$6.IN_1
- net V_LS_1: now also IC1.28
- net V_LS_2: now also IC1.29
- net V_LS_3: now also IC1.30
- net V_LS_4: now also IC1.31
- net XSHUT3: now also IC1.38; no longer IC1.33
- net XSHUT5: now also IC1.79
Routing:
- net +3.3V: track 9.54 -> 251.5 mm, vias 14 -> 39
- net V_LS_2: track 0.00 -> 95.6 mm, vias 0 -> 6
- net V_LS_4: track 0.00 -> 91.8 mm, vias 0 -> 4
- net TOF_GPIO5: track 0.00 -> 66.8 mm, vias 0 -> 1
- net XSHUT5: track 0.00 -> 64.9 mm, vias 0 -> 1
- net V_LS_3: track 0.00 -> 61.7 mm, vias 0 -> 3
- net V_LS_1: track 0.00 -> 46.9 mm
- net 5V_SW: track 0.00 -> 31.9 mm, vias 0 -> 4
- net SWO: track 0.00 -> 22.4 mm, vias 0 -> 3
- net V_BAT: track 0.00 -> 5.98 mm
- net N$11: track 0.00 -> 5.95 mm
- net N$10: track 0.00 -> 4.26 mm, vias 0 -> 1
- net VCP_RX: track 9.87 -> 13.4 mm
- net N$6: track 0.00 -> 3.18 mm, vias 0 -> 1
- net N$9: track 0.00 -> 3.10 mm, vias 0 -> 1
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- added copper zone on layer 2, net +3.3V
- added copper zone on layer 15, net GND
- added copper zone on layer 2, net GND

Commit message: 07_11_2021_23_28
Parts:
- added R12, R13, R14: 10k, rcl:R0402
- added SV7: (no value), con-lstb:MA03-1
- added U$7: BAT_POW, SamacSys_Parts:BAT_POW
- R1, R11, R3, R5, R7, R9: value (none) -> 10k
- R10, R4, R6, R8: value (none) -> 200
- R2: value (none) -> 25
- U$6: device SamacSys_Parts:MD_OUT -> SamacSys_Parts:BAT_POW
- moved U$5 6.99 mm to (5.71, 15.7)
- moved U$4 5.92 mm to (65.7, 78.2)
- moved SV2 0.38 mm to (3.05, 47.2)
Connections:
- new net START_SW: IC1.34, SV7.1
- net +3.3V: now also R12.2, R13.1, R14.2, SV7.3
- net 5V_SW: now also U$7.P$1
- net GND: now also SV7.2, U$6.P$2, U$7.P$2; no longer U$6.IN_2
- net MD_DIS1: now also R13.2
- net MD_DIS2: now also R14.1
- net MD_NDIS: now also R12.1
- net V_BAT: now also U$6.P$1; no longer U$6.IN_1
Routing:
- net +3.3V: track 251.5 -> 261.3 mm, vias 39 -> 40
- net START_SW: track 0.00 -> 9.77 mm, vias 0 -> 1
- net 5V_SW: track 31.9 -> 39.9 mm
- net TOF_SCL: track 304.2 -> 300.2 mm
- net MD_DIS2: track 19.9 -> 23.7 mm
- net MD_NDIS: track 18.6 -> 21.9 mm
- net TOF_SDA: track 303.6 -> 305.5 mm
- net MD_DIS1: track 12.5 -> 13.4 mm
- net V_LS_4: track 91.8 -> 91.2 mm
- net V_LS_3: track 61.7 -> 62.3 mm
- net GND: vias 23 -> 58

Commit message: final
Parts:
- added 3V3, GND, IBUS_RX: (no value), wirepad:SMD1,27-2,54
- added SJ2: (no value), jumper:SJ_2
- added SV8: (no value), con-lstb:MA03-1
- R2: value 25 -> 51
- SV7: device con-lstb:MA03-1 -> con-lstb:MA04-1
Connections:
- new net IBUS_RX: IBUS_RX.1, SJ2.2
- new net KILL_SW: SV7.1, SV8.1
- new net RX: IC1.37, SJ2.1
- new net S_WIRE: IC1.38, SJ2.3
- net +3.3V: now also 3V3.1, SV7.4; no longer SV7.3
- net 5V_SW: now also SV8.2
- net GND: now also GND.1, SV7.3, SV8.3; no longer SV7.2
- net START_SW: now also SV7.2; no longer SV7.1
- net TOF_GPIO3: now also IC1.39; no longer IC1.37
- net XSHUT3: now also IC1.40; no longer IC1.38
Routing:
- net 5V_SW: track 39.9 -> 101.0 mm
- net IBUS_RX: track 0.00 -> 7.06 mm
- net RX: track 0.00 -> 6.82 mm, vias 0 -> 1
- net S_WIRE: track 0.00 -> 6.29 mm, vias 0 -> 1
- net KILL_SW: track 0.00 -> 5.75 mm
- net +3.3V: track 261.3 -> 265.3 mm
Other:
- board text added: "RX"
- board text added: "TX"
