File: Minisumo_V1.sch (EAGLE design)
At the start: 57 parts, among them IC1 STM32H743VIT6NORMAL, J1 FTSH-107-01-L-DV-K-TR, Y1 ECS-3225MV

Commit message: 07_11_2021_15_50
Connections:
- net MD_CS1: now also IC1.PA9
- net MD_CS2: now also IC1.PD11
- net MD_DIS1: now also IC1.PA8
- net MD_DIS2: now also IC1.PD12
- net MD_IN1_PWM_A: now also IC1.PC6
- net MD_IN1_PWM_B: now also IC1.PD14
- net MD_IN2_DIR_A: now also IC1.PC7
- net MD_IN2_DIR_B: now also IC1.PD13
- net MD_NDIS: now also IC1.PD15
Changed lines of the file:
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@@
+</segment>
+</net>
+<net name="MD_CS1" class="0">
+<segment>
+<pinref part="IC1" gate="G$1" pin="PA9"/>
+<wire x1="121.92" y1="58.42" x2="127" y2="58.42" width="0.1524" layer="91"/>
+<label x="127" y="58.42" size="1.27" layer="95" xref="yes"/>
+</segment>
+</net>
+<net name="MD_NDIS" class="0">
+<segment>
+<pinref part="IC1" gate="G$1" pin="PD15"/>
+<wire x1="121.92" y1="43.18" x2="127" y2="43.18" width="0.1524" layer="91"/>
+<label x="127" y="43.18" size="1.27" layer="95" xref="yes"/>
+</segment>
+</net>
+<net name="MD_CS2" class="0">
+<segment>
+<pinref part="IC1" gate="G$1" pin="PD11"/>
+<wire x1="121.92" y1="33.02" x2="127" y2="33.02" width="0.1524" layer="91"/>
+<label x="127" y="33.02" size="1.27" layer="95" xref="yes"/>
+</segment>
+</net>
+<net name="MD_DIS1" class="0">
+<segment>
+<pinref part="IC1" gate="G$1" pin="PA8"/>
+<wire x1="121.92" y1="55.88" x2="127" y2="55.88" width="0.1524" layer="91"/>
+<label x="127" y="55.88" size="1.27" layer="95" xref="yes"/>
+</segment>
+</net>
+<net name="MD_DIS2" class="0">
+<segment>
+<pinref part="IC1" gate="G$1" pin="PD12"/>
+<wire x1="121.92" y1="35.56" x2="127" y2="35.56" width="0.1524" layer="91"/>
+<label x="127" y="35.56" size="1.27" layer="95" xref="yes"/>
+</segment>
+</net>
+<net name="MD_IN1_PWM_A" class="0">
+<segment>
+<pinref part="IC1" gate="G$1" pin="PC6"/>
+<wire x1="121.92" y1="45.72" x2="127" y2="50.8" width="0.1524" layer="91"/>
+<label x="127" y="50.8" size="1.27" layer="95" xref="yes"/>
+</segment>
+</net>
+<net name="MD_IN2_DIR_A" class="0">
+<segment>
+<pinref part="IC1" gate="G$1" pin="PC7"/>
+<wire x1="121.92" y1="48.26" x2="127" y2="53.34" width="0.1524" layer="91"/>
+<label x="127" y="53.34" size="1.27" layer="95" xref="yes"/>
+</segment>
+</net>
+<net name="MD_IN1_PWM_B" class="0">
+<segment>
+<pinref part="IC1" gate="G$1" pin="PD14"/>
+<wire x1="121.92" y1="40.64" x2="127" y2="40.64" width="0.1524" layer="91"/>
+<label x="127" y="40.64" size="1.27" layer="95" xref="yes"/>
+</segment>
+</net>
+<net name="MD_IN2_DIR_B" class="0">
+<segment>
+<pinref part="IC1" gate="G$1" pin="PD13"/>
+<wire x1="121.92" y1="38.1" x2="127" y2="38.1" width="0.1524" layer="91"/>
+<label x="127" y="38.1" size="1.27" layer="95" xref="yes"/>
 </segment>
 </net>

Commit message: 07_11_2021_22_21
Parts:
- added U$4, U$5: MD_OUT, SamacSys_Parts:MD_OUT
- added U$6: BAT_POW, SamacSys_Parts:BAT_POW
Connections:
- net GND: now also U$6.GND
- net MD_OUT1A: now also U$4.IN_1
- net MD_OUT1B: now also U$5.IN_1
- net MD_OUT2A: now also U$4.IN_2
- net MD_OUT2B: now also U$5.IN_2
- net TOF_GPIO3: now also IC1.PE7; no longer IC1.PC4
- net TOF_GPIO5: now also IC1.PC10
- net V_BAT: now also U$6.BAT+
- net V_LS_1: now also IC1.PA4
- net V_LS_2: now also IC1.PA5
- net V_LS_3: now also IC1.PA6
- net V_LS_4: now also IC1.PA7
- net XSHUT3: now also IC1.PE8; no longer IC1.PC5
- net XSHUT5: now also IC1.PC11
Changed lines of the file:
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@@
 </part>
 <part name="FRAME2" library="frames" library_urn="urn:adsk.eagle:library:229" deviceset="A4L-LOC" device=""/>
-<part name="SV1" library="con-lstb" library_urn="urn:adsk.eagle:library:162" deviceset="MA07-1" device="" package3d_urn="urn:adsk.eagle:package:8341/1"/>
+<part name="SV1" library="con-lstb" deviceset="MA07-1" device="" package3d_urn="urn:adsk.eagle:package:8341/1"/>
 <part name="SV2" library="con-lstb" library_urn="urn:adsk.eagle:library:162" deviceset="MA07-1" device="" package3d_urn="urn:adsk.eagle:package:8341/1"/>
 <part name="SV3" library="con-lstb" library_urn="urn:adsk.eagle:library:162" deviceset="MA07-1" device="" package3d_urn="urn:adsk.eagle:package:8341/1"/>
@@
 <part name="SUPPLY40" library="Power_Symbols" library_urn="urn:adsk.eagle:library:16502351" deviceset="+3.3V" device="" value="+3.3V"/>
 <part name="SUPPLY41" library="Power_Symbols" library_urn="urn:adsk.eagle:library:16502351" deviceset="+3.3V" device="" value="+3.3V"/>
+<part name="U$4" library="SamacSys_Parts" deviceset="MD_OUT" device=""/>
+<part name="U$5" library="SamacSys_Parts" deviceset="MD_OUT" device=""/>
+<part name="U$6" library="SamacSys_Parts" deviceset="BAT_POW" device=""/>
+<part name="GND15" library="supply1" library_urn="urn:adsk.eagle:library:371" deviceset="GND" device=""/>
 </parts>
 <sheets>
@@
 </sheet>
 <sheet>
-<description>MCU Power</description>
+<description>Power</description>
 <plain>
 </plain>
@@
 <attribute name="NAME" x="74.168" y="42.418" size="2" layer="95"/>
 <attribute name="VALUE" x="74.168" y="37.846" size="2" layer="96"/>
+</instance>
+<instance part="U$6" gate="G$1" x="71.12" y="-15.24" smashed="yes"/>
+<instance part="GND15" gate="1" x="91.44" y="-27.94" smashed="yes">
+<attribute name="VALUE" x="88.9" y="-30.48" size="1.778" layer="96"/>
 </instance>
 </instances>
@@
 <junction x="83.82" y="30.48"/>
 </segment>
+<segment>
+<pinref part="U$6" gate="G$1" pin="GND"/>
+<wire x1="86.36" y1="-20.32" x2="91.44" y2="-20.32" width="0.1524" layer="91"/>
+<wire x1="91.44" y1="-20.32" x2="91.44" y2="-25.4" width="0.1524" layer="91"/>
+<pinref part="GND15" gate="1" pin="GND"/>
+</segment>
 </net>
 <net name="5V_SW" class="0">
@@
 </segment>
 </net>
+<net name="V_BAT" class="0">
+<segment>
+<pinref part="U$6" gate="G$1" pin="BAT+"/>
+<wire x1="86.36" y1="0" x2="93.98" y2="0" width="0.1524" layer="91"/>
+<label x="93.98" y="0" size="1.27" layer="95" xref="yes"/>
+</segment>
+</net>
 </nets>
 </sheet>
@@
 <attribute name="VALUE" x="20.32" y="30.48" size="1.778" layer="96"/>
 </instance>
-<instance part="GND4" gate="1" x="53.34" y="-12.7" smashed="yes">
-<attribute name="VALUE" x="50.8" y="-15.24" size="1.778" layer="96"/>
+<instance part="GND4" gate="1" x="45.72" y="-5.08" smashed="yes">
+<attribute name="VALUE" x="43.18" y="-7.62" size="1.778" layer="96"/>
 </instance>
 <instance part="GND5" gate="1" x="114.3" y="-15.24" smashed="yes" rot="R90">
 <attribute name="VALUE" x="116.84" y="-17.78" size="1.778" layer="96" rot="R90"/>
 </instance>
-<instance part="SUPPLY2" gate="G$1" x="55.88" y="-7.62" smashed="yes" rot="R180">
-<attribute name="VALUE" x="56.007" y="-10.668" size="1.778" layer="96" rot="R180" align="bottom-center"/>
+<instance part="SUPPLY2" gate="G$1" x="55.88" y="-20.32" smashed="yes" rot="R180">
+<attribute name="VALUE" x="56.007" y="-20.828" size="1.778" layer="96" rot="R180" align="bottom-center"/>
 </instance>
 <instance part="SUPPLY3" gate="G$1" x="114.3" y="-5.08" smashed="yes" rot="R180">
@@
 <segment>
 <pinref part="IC1" gate="G$1" pin="VSS_2"/>
-<wire x1="53.34" y1="-2.54" x2="53.34" y2="-10.16" width="0.1524" layer="91"/>
+<wire x1="53.34" y1="-2.54" x2="45.72" y2="-2.54" width="0.1524" layer="91"/>
 <pinref part="GND4" gate="1" pin="GND"/>
 </segment>
@@
 <segment>
 <pinref part="IC1" gate="G$1" pin="VDD_2"/>
-<wire x1="55.88" y1="-2.54" x2="55.88" y2="-7.62" width="0.1524" layer="91"/>
+<wire x1="55.88" y1="-2.54" x2="55.88" y2="-20.32" width="0.1524" layer="91"/>
 <pinref part="SUPPLY2" gate="G$1" pin="+3.3V"/>
 </segment>
@@
 <net name="TOF_GPIO3" class="0">
 <segment>
-<label x="68.58" y="-10.16" size="1.27" layer="95" rot="R270" xref="yes"/>
-<pinref part="IC1" gate="G$1" pin="PC4"/>
-<wire x1="68.58" y1="-2.54" x2="68.58" y2="-10.16" width="0.1524" layer="91"/>
+<label x="81.28" y="-10.16" size="1.27" layer="95" rot="R270" xref="yes"/>
+<pinref part="IC1" gate="G$1" pin="PE7"/>
+<wire x1="81.28" y1="-10.16" x2="81.28" y2="-2.54" width="0.1524" layer="91"/>
 </segment>
 </net>
@@
 <net name="XSHUT3" class="0">
 <segment>
-<label x="71.12" y="-10.16" size="1.27" layer="95" rot="R270" xref="yes"/>
-<pinref part="IC1" gate="G$1" pin="PC5"/>
-<wire x1="71.12" y1="-10.16" x2="71.12" y2="-2.54" width="0.1524" layer="91"/>
+<label x="83.82" y="-10.16" size="1.27" layer="95" rot="R270" xref="yes"/>
+<wire x1="83.82" y1="-10.16" x2="83.82" y2="-2.54" width="0.1524" layer="91"/>
+<pinref part="IC1" gate="G$1" pin="PE8"/>
 </segment>
 </net>
@@
 <segment>
 <pinref part="IC1" gate="G$1" pin="PC6"/>
-<wire x1="121.92" y1="45.72" x2="127" y2="50.8" width="0.1524" layer="91"/>
-<label x="127" y="50.8" size="1.27" layer="95" xref="yes"/>
+<wire x1="121.92" y1="45.72" x2="127" y2="45.72" width="0.1524" layer="91"/>
+<label x="127" y="45.72" size="1.27" layer="95" xref="yes"/>
 </segment>
 </net>
@@
 <segment>
 <pinref part="IC1" gate="G$1" pin="PC7"/>
-<wire x1="121.92" y1="48.26" x2="127" y2="53.34" width="0.1524" layer="91"/>
-<label x="127" y="53.34" size="1.27" layer="95" xref="yes"/>
+<wire x1="121.92" y1="48.26" x2="127" y2="48.26" width="0.1524" layer="91"/>
+<label x="127" y="48.26" size="1.27" layer="95" xref="yes"/>
 </segment>
 </net>
@@
 <wire x1="121.92" y1="38.1" x2="127" y2="38.1" width="0.1524" layer="91"/>
 <label x="127" y="38.1" size="1.27" layer="95" xref="yes"/>
+</segment>
+</net>
+<net name="XSHUT5" class="0">
+<segment>
+<pinref part="IC1" gate="G$1" pin="PC11"/>
+<wire x1="106.68" y1="93.98" x2="106.68" y2="96.52" width="0.1524" layer="91"/>
+<label x="106.68" y="96.52" size="1.27" layer="95" rot="R90" xref="yes"/>
+</segment>
+</net>
+<net name="TOF_GPIO5" class="0">
+<segment>
+<pinref part="IC1" gate="G$1" pin="PC10"/>
+<wire x1="109.22" y1="93.98" x2="109.22" y2="96.52" width="0.1524" layer="91"/>
+<label x="109.22" y="96.52" size="1.27" layer="95" rot="R90" xref="yes"/>
+</segment>
+</net>
+<net name="V_LS_1" class="0">
+<segment>
+<pinref part="IC1" gate="G$1" pin="PA4"/>
+<wire x1="58.42" y1="-2.54" x2="58.42" y2="-5.08" width="0.1524" layer="91"/>
+<label x="58.42" y="-5.08" size="1.27" layer="95" rot="R270" xref="yes"/>
+</segment>
+</net>
+<net name="V_LS_2" class="0">
+<segment>
+<pinref part="IC1" gate="G$1" pin="PA5"/>
+<wire x1="60.96" y1="-2.54" x2="60.96" y2="-5.08" width="0.1524" layer="91"/>
+<label x="60.96" y="-5.08" size="1.27" layer="95" rot="R270" xref="yes"/>
+</segment>
+</net>
+<net name="V_LS_3" class="0">
+<segment>
+<pinref part="IC1" gate="G$1" pin="PA6"/>
+<wire x1="63.5" y1="-2.54" x2="63.5" y2="-5.08" width="0.1524" layer="91"/>
+<label x="63.5" y="-5.08" size="1.27" layer="95" rot="R270" xref="yes"/>
+</segment>
+</net>
+<net name="V_LS_4" class="0">
+<segment>
+<pinref part="IC1" gate="G$1" pin="PA7"/>
+<wire x1="66.04" y1="-2.54" x2="66.04" y2="-5.08" width="0.1524" layer="91"/>
+<label x="66.04" y="-5.08" size="1.27" layer="95" rot="R270" xref="yes"/>
 </segment>
 </net>
@@
 <attribute name="VALUE" x="106.553" y="61.468" size="1.778" layer="96" align="bottom-center"/>
 </instance>
+<instance part="U$4" gate="G$1" x="-5.08" y="101.6" smashed="yes"/>
+<instance part="U$5" gate="G$1" x="119.38" y="101.6" smashed="yes"/>
 </instances>
 <busses>
@@
 <label x="81.28" y="50.8" size="1.27" layer="95" xref="yes"/>
 </segment>
+<segment>
+<pinref part="U$5" gate="G$1" pin="IN_1"/>
+<wire x1="99.06" y1="101.6" x2="88.9" y2="101.6" width="0.1524" layer="91"/>
+<label x="88.9" y="101.6" size="1.27" layer="95" rot="R180" xref="yes"/>
+</segment>
 </net>
 <net name="MD_OUT2B" class="0">
@@
 <label x="35.56" y="40.64" size="1.27" layer="95" rot="R180" xref="yes"/>
 </segment>
+<segment>
+<pinref part="U$5" gate="G$1" pin="IN_2"/>
+<wire x1="139.7" y1="101.6" x2="139.7" y2="91.44" width="0.1524" layer="91"/>
+<label x="139.7" y="91.44" size="1.27" layer="95" rot="R270" xref="yes"/>
+</segment>
 </net>
 <net name="MD_OUT1A" class="0">
@@
 <label x="35.56" y="73.66" size="1.27" layer="95" rot="R180" xref="yes"/>
 </segment>
+<segment>
+<pinref part="U$4" gate="G$1" pin="IN_1"/>
+<wire x1="-25.4" y1="101.6" x2="-25.4" y2="86.36" width="0.1524" layer="91"/>
+<label x="-25.4" y="86.36" size="1.27" layer="95" rot="R270" xref="yes"/>
+<label x="-25.4" y="86.36" size="1.27" layer="95" rot="R270" xref="yes"/>
+</segment>
 </net>
 <net name="MD_OUT2A" class="0">
@@
 <label x="81.28" y="81.28" size="1.27" layer="95" xref="yes"/>
 </segment>
-</net>
+<segment>
+<pinref part="U$4" gate="G$1" pin="IN_2"/>
+<wire x1="15.24" y1="101.6" x2="20.32" y2="101.6" width="0.1524" layer="91"/>
+<label x="20.32" y="101.6" size="1.27" layer="95" xref="yes"/>
+</segment>
+</net>

Commit message: 07_11_2021_23_28
Parts:
- added R12, R13, R14: 10k, rcl:R-EU_R0402
- added SV7: (no value), con-lstb:MA03-1
- added U$7: BAT_POW, SamacSys_Parts:BAT_POW
- R1, R11, R3, R5, R7, R9: value (none) -> 10k
- R10, R4, R6, R8: value (none) -> 200
- R2: value (none) -> 25
Connections:
- new net START_SW: IC1.PB0, SV7.1
- net +3.3V: now also R12.2, R13.1, R14.2, SV7.3
- net 5V_SW: now also U$7.BAT+
- net GND: now also SV7.2, U$7.GND
- net MD_DIS1: now also R13.2
- net MD_DIS2: now also R14.1
- net MD_NDIS: now also R12.1

Commit message: final
Parts:
- added 3V3, GND, IBUS_RX: (no value), wirepad:SMD2
- added SJ2: (no value), jumper:SJ2W
- added SV8: (no value), con-lstb:MA03-1
- R2: value 25 -> 51
- SV7: device con-lstb:MA03-1 -> con-lstb:MA04-1
Connections:
- new net IBUS_RX: IBUS_RX.P, SJ2.2
- new net KILL_SW: SV7.1, SV8.1
- new net RX: IC1.PE7, SJ2.1
- new net S_WIRE: IC1.PE8, SJ2.3
- net +3.3V: now also 3V3.P, SV7.4; no longer SV7.3
- net 5V_SW: now also SV8.2
- net GND: now also GND.P, SV7.3, SV8.3; no longer SV7.2
- net START_SW: now also SV7.2; no longer SV7.1
- net TOF_GPIO3: now also IC1.PE9; no longer IC1.PE7
- net XSHUT3: now also IC1.PE10; no longer IC1.PE8
